File: hardware/PC_Interface_Card/PC_Interface_Card.kicad_sch (KiCad schematic)
At the start: 79 parts, among them J1 GSB1C41110SSHR, J2 DM3BT-DSF-PEJS, J3 BM11B-GHS-TBT, J4 GHR-11V-S, J5 GHR-11V-S, SW1 CherryMX, SW2 CherryMX, SW3 CherryMX, SW4 CherryMX, SW5 CherryMX, SW6 TL1240YQ2JBLK, SW7 TL1240YQ2JBLK, SW8 TL1240YQ2JBLK, U1 USBLC6-2SC6, U2 TLV1117LV33DCYR, U3 MB85RS4MTYPN-GS-AWEWE1, U4 ESP32-S3-WROOM-1

Commit message: Added via and trace rules
Connections:
- net SW_EN: no longer C14.1, R25.1, SW6.1, SW6.2
- net SW_PLAY: now reaches U4.36 (RXD0)
- net SW_PLAY: now also C14.1, R25.1, SW6.1, SW6.2
- no-connect marks 16 -> 15
Changed lines of the file:
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@@
 	)
 	(no_connect
-		(at 467.36 74.93)
-	)
-	(no_connect
 		(at 467.36 87.63)
 	)
@@
 	(wire
 		(pts
+			(xy 467.36 74.93) (xy 472.44 74.93)
+		)
+		(stroke
+			(width 0)
+			(type default)
+		)
+	)
+	(wire
+		(pts
 			(xy 128.27 201.93) (xy 128.27 207.01)
 		)
@@
 		)
 	)
+	(global_label "SW_PLAY"
+		(shape bidirectional)
+		(at 472.44 74.93 0)
+		(fields_autoplaced yes)
+		(effects
+			(font
+				(size 1.27 1.27)
+			)
+			(justify left)
+		)
+		(property "Intersheetrefs" "${INTERSHEET_REFS}"
+			(at 484.6403 74.93 0)
+			(effects
+				(font
+					(size 1.27 1.27)
+				)
+				(justify left)
+				(hide yes)
+			)
+		)
+	)
 	(global_label "CS_DISP"
 		(shape bidirectional)
@@
 		)
 	)
+	(global_label "SW_PLAY"
+		(shape bidirectional)
+		(at 360.68 189.23 180)
+		(fields_autoplaced yes)
+		(effects
+			(font
+				(size 1.27 1.27)
+			)
+			(justify right)
+		)
+		(property "Intersheetrefs" "${INTERSHEET_REFS}"
+			(at 348.4797 189.23 0)
+			(effects
+				(font
+					(size 1.27 1.27)
+				)
+				(justify right)
+				(hide yes)
+			)
+		)
+	)
 	(global_label "SW_EN"
 		(shape bidirectional)
@@
 			(effects
 				(font
-					(size 1.27 1.27)
-				)
-				(justify right)
-				(hide yes)
-			)
-		)
-	)
-	(global_label "SW_EN"
-		(shape bidirectional)
-		(at 360.68 189.23 180)
-		(fields_autoplaced yes)
-		(effects
-			(font
-				(size 1.27 1.27)
-			)
-			(justify right)
-		)
-		(property "Intersheetrefs" "${INTERSHEET_REFS}"
-			(at 350.4755 189.23 0)
-			(effects
-				(font
