File: hardware/PC_Interface_Card/_autosave-PC_Interface_Card.kicad_pcb (KiCad board)
At the start: 2 copper layers, 91.9 x 72 mm, 84 parts, among them J1 GSB1C41110SSHR, J2 DM3BT-DSF-PEJS, J4 BM11B-GHS-TBT, SW1 CherryMX, SW2 CherryMX, SW3 CherryMX, SW4 CherryMX, SW5 CherryMX, SW6 TL1240YQ2JBLK, SW7 SW_Push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

Commit message: Fixes on the layout for refab due to my copyrighted SMD vias
Routing:
- net D-: track 54.9 -> 52.9 mm
- net D+: track 54.9 -> 52.9 mm
- net D0_SDMMC: track 55.2 -> 53.9 mm
- net SW_LEFT: track 66.9 -> 65.7 mm
- net ENC_A: track 47.7 -> 46.5 mm
- net MOSI: track 68.5 -> 69.5 mm
- net SW_PLAY: track 55.3 -> 54.5 mm
- net (no net): vias 0 -> 1
